File: kicad/AXIS_SENSOR.sch (KiCad schematic (older format))
At the start: 4 parts, among them U8 MPU6500

Commit message: 徐々に部品を配置，部品の確認
Parts:
- renumbered C30 to C29, C31 to C30, C32 to C31
Changed lines of the file:
@@
 $EndDescr
 $Comp
-L +3.3V #PWR086
+L +3.3V #PWR085
 U 1 1 57CCAAD0
 P 5700 2700
-F 0 "#PWR086" H 5700 2550 50  0001 C CNN
+F 0 "#PWR085" H 5700 2550 50  0001 C CNN
 F 1 "+3.3V" H 5750 2850 50  0000 C CNN
 F 2 "" H 5700 2700 50  0000 C CNN
@@
 	5700 2700 5700 3200
 $Comp
-L GND #PWR087
+L GND #PWR086
 U 1 1 57CCAAFB
 P 5500 4700
-F 0 "#PWR087" H 5500 4450 50  0001 C CNN
+F 0 "#PWR086" H 5500 4450 50  0001 C CNN
 F 1 "GND" H 5500 4550 50  0000 C CNN
 F 2 "" H 5500 4700 50  0000 C CNN
@@
 AXIS_MISO
 $Comp
-L GND #PWR088
+L GND #PWR087
 U 1 1 57CCAB79
 P 6400 4700
-F 0 "#PWR088" H 6400 4450 50  0001 C CNN
+F 0 "#PWR087" H 6400 4450 50  0001 C CNN
 F 1 "GND" H 6400 4550 50  0000 C CNN
 F 2 "" H 6400 4700 50  0000 C CNN
@@
 	6400 3700 6300 3700
 $Comp
-L C C32
+L C C31
 U 1 1 57CCABB6
 P 7200 3950
-F 0 "C32" H 7225 4050 50  0000 L CNN
+F 0 "C31" H 7225 4050 50  0000 L CNN
 F 1 "0.1u" H 7225 3850 50  0000 L CNN
 F 2 "Capacitors_SMD:C_0402" H 7238 3800 50  0001 C CNN
@@
 	7200 3600 6300 3600
 $Comp
-L GND #PWR089
+L GND #PWR088
 U 1 1 57CCAC2E
 P 7200 4700
-F 0 "#PWR089" H 7200 4450 50  0001 C CNN
+F 0 "#PWR088" H 7200 4450 50  0001 C CNN
 F 1 "GND" H 7200 4550 50  0000 C CNN
 F 2 "" H 7200 4700 50  0000 C CNN
@@
 	6500 4400 6300 4400
 $Comp
-L GND #PWR090
+L GND #PWR089
 U 1 1 57CCB3DF
 P 5100 3000
-F 0 "#PWR090" H 5100 2750 50  0001 C CNN
+F 0 "#PWR089" H 5100 2750 50  0001 C CNN
 F 1 "GND" H 5100 2850 50  0000 C CNN
 F 2 "" H 5100 3000 50  0000 C CNN
@@
 $EndComp
 $Comp
-L +3.3V #PWR091
+L +3.3V #PWR090
 U 1 1 57CCB773
 P 5500 2700
-F 0 "#PWR091" H 5500 2550 50  0001 C CNN
+F 0 "#PWR090" H 5500 2550 50  0001 C CNN
 F 1 "+3.3V" H 5450 2850 50  0000 C CNN
 F 2 "" H 5500 2700 50  0000 C CNN
@@
 	5100 2900 5200 2900
 $Comp
-L C_Small C30
+L C_Small C29
 U 1 1 57CCB95E
 P 5300 2900
-F 0 "C30" H 5310 2970 50  0000 L CNN
+F 0 "C29" H 5310 2970 50  0000 L CNN
 F 1 "0.01u" H 5310 2820 50  0000 L CNN
 F 2 "Capacitors_SMD:C_0402" H 5300 2900 50  0001 C CNN
@@
 $EndComp
 $Comp
-L C_Small C31
+L C_Small C30
 U 1 1 57CCB9B9
 P 5900 2900
-F 0 "C31" H 5910 2970 50  0000 L CNN
+F 0 "C30" H 5910 2970 50  0000 L CNN
 F 1 "0.1u" H 5910 2820 50  0000 L CNN
 F 2 "Capacitors_SMD:C_0402" H 5900 2900 50  0001 C CNN
@@
 	5800 2900 5700 2900
 $Comp
-L GND #PWR092
+L GND #PWR091
 U 1 1 57CCBA56
 P 6100 3000
-F 0 "#PWR092" H 6100 2750 50  0001 C CNN
+F 0 "#PWR091" H 6100 2750 50  0001 C CNN
 F 1 "GND" H 6100 2850 50  0000 C CNN
 F 2 "" H 6100 3000 50  0000 C CNN

Commit message: リポ充電基板を追加
Connections:
- net AXIS_CAP: now reaches C31.1, U8.10 (REGOUT)
Changed lines of the file:
@@
 $Descr A4 11693 8268
 encoding utf-8
-Sheet 11 13
+Sheet 11 14
 Title ""
 Date ""
@@
 Text Notes 4200 2400 0    100  ~ 0
 AXIS Sensor
+Text Label 7200 3600 0    60   ~ 0
+AXIS_CAP
 $EndSCHEMATC
