File: kicad/AXIS_SENSOR.sch (KiCad schematic (older format))
At the start: 4 parts, among them U8 MPU6500

Commit message: 自動配線用にdsn吐き出し
Parts:
- renumbered C29 to C26, C30 to C27, C31 to C28, U8 to U7
Changed lines of the file:
@@
 $EndDescr
 $Comp
-L +3.3V #PWR085
+L +3.3V #PWR081
 U 1 1 57CCAAD0
 P 5700 2700
-F 0 "#PWR085" H 5700 2550 50  0001 C CNN
+F 0 "#PWR081" H 5700 2550 50  0001 C CNN
 F 1 "+3.3V" H 5750 2850 50  0000 C CNN
 F 2 "" H 5700 2700 50  0000 C CNN
@@
 	5700 2700 5700 3200
 $Comp
-L GND #PWR086
+L GND #PWR082
 U 1 1 57CCAAFB
 P 5500 4700
-F 0 "#PWR086" H 5500 4450 50  0001 C CNN
+F 0 "#PWR082" H 5500 4450 50  0001 C CNN
 F 1 "GND" H 5500 4550 50  0000 C CNN
 F 2 "" H 5500 4700 50  0000 C CNN
@@
 AXIS_MISO
 $Comp
-L GND #PWR087
+L GND #PWR083
 U 1 1 57CCAB79
 P 6400 4700
-F 0 "#PWR087" H 6400 4450 50  0001 C CNN
+F 0 "#PWR083" H 6400 4450 50  0001 C CNN
 F 1 "GND" H 6400 4550 50  0000 C CNN
 F 2 "" H 6400 4700 50  0000 C CNN
@@
 	6400 3700 6300 3700
 $Comp
-L C C31
+L C C28
 U 1 1 57CCABB6
 P 7200 3950
-F 0 "C31" H 7225 4050 50  0000 L CNN
+F 0 "C28" H 7225 4050 50  0000 L CNN
 F 1 "0.1u" H 7225 3850 50  0000 L CNN
 F 2 "Capacitors_SMD:C_0402" H 7238 3800 50  0001 C CNN
@@
 	7200 3600 6300 3600
 $Comp
-L GND #PWR088
+L GND #PWR084
 U 1 1 57CCAC2E
 P 7200 4700
-F 0 "#PWR088" H 7200 4450 50  0001 C CNN
+F 0 "#PWR084" H 7200 4450 50  0001 C CNN
 F 1 "GND" H 7200 4550 50  0000 C CNN
 F 2 "" H 7200 4700 50  0000 C CNN
@@
 	6500 4400 6300 4400
 $Comp
-L GND #PWR089
+L GND #PWR085
 U 1 1 57CCB3DF
 P 5100 3000
-F 0 "#PWR089" H 5100 2750 50  0001 C CNN
+F 0 "#PWR085" H 5100 2750 50  0001 C CNN
 F 1 "GND" H 5100 2850 50  0000 C CNN
 F 2 "" H 5100 3000 50  0000 C CNN
@@
 $EndComp
 $Comp
-L MPU6500 U8
+L MPU6500 U7
 U 1 1 57CCB62A
 P 5700 3650
-F 0 "U8" H 5250 4050 50  0000 C CNN
+F 0 "U7" H 5250 4050 50  0000 C CNN
 F 1 "MPU6500" H 6000 4050 50  0000 C CNN
 F 2 "mouse:QFN-24-1EP_3x3mm_Pitch0.4mm" H 5100 2650 50  0001 C CNN
@@
 $EndComp
 $Comp
-L +3.3V #PWR090
+L +3.3V #PWR086
 U 1 1 57CCB773
 P 5500 2700
-F 0 "#PWR090" H 5500 2550 50  0001 C CNN
+F 0 "#PWR086" H 5500 2550 50  0001 C CNN
 F 1 "+3.3V" H 5450 2850 50  0000 C CNN
 F 2 "" H 5500 2700 50  0000 C CNN
@@
 	5100 2900 5200 2900
 $Comp
-L C_Small C29
+L C_Small C26
 U 1 1 57CCB95E
 P 5300 2900
-F 0 "C29" H 5310 2970 50  0000 L CNN
+F 0 "C26" H 5310 2970 50  0000 L CNN
 F 1 "0.01u" H 5310 2820 50  0000 L CNN
 F 2 "Capacitors_SMD:C_0402" H 5300 2900 50  0001 C CNN
@@
 $EndComp
 $Comp
-L C_Small C30
+L C_Small C27
 U 1 1 57CCB9B9
 P 5900 2900
-F 0 "C30" H 5910 2970 50  0000 L CNN
+F 0 "C27" H 5910 2970 50  0000 L CNN
 F 1 "0.1u" H 5910 2820 50  0000 L CNN
 F 2 "Capacitors_SMD:C_0402" H 5900 2900 50  0001 C CNN
@@
 	5800 2900 5700 2900
 $Comp
-L GND #PWR091
+L GND #PWR087
 U 1 1 57CCBA56
 P 6100 3000
-F 0 "#PWR091" H 6100 2750 50  0001 C CNN
+F 0 "#PWR087" H 6100 2750 50  0001 C CNN
 F 1 "GND" H 6100 2850 50  0000 C CNN
 F 2 "" H 6100 3000 50  0000 C CNN
