File: kicad/IR_LED.sch (KiCad schematic (older format))
At the start: 5 parts, among them Q2 IRFML8244

Commit message: フットプリント調整
Changed lines of the file:
@@
 AR Path="/57CEFE78/57CF03B8" Ref="Q2"  Part="1"
 AR Path="/57CF2D36/57CF03B8" Ref="Q3"  Part="1"
-F 0 "Q3" H 6100 4850 50  0000 R CNN
+F 0 "Q2" H 6100 4850 50  0000 R CNN
 F 1 "IRFML8244" H 6450 4750 50  0000 R CNN
 F 2 "TO_SOT_Packages_SMD:SOT-23" H 6000 4900 50  0001 C CNN
@@
 AR Path="/57CEFE78/57CF03C0" Ref="#PWR060"  Part="1"
 AR Path="/57CF2D36/57CF03C0" Ref="#PWR083"  Part="1"
-F 0 "#PWR083" H 5900 5050 50  0001 C CNN
+F 0 "#PWR060" H 5900 5050 50  0001 C CNN
 F 1 "GND" H 5900 5150 50  0000 C CNN
 F 2 "" H 5900 5300 50  0000 C CNN
@@
 AR Path="/57CEFE78/57CF03DE" Ref="D3"  Part="1"
 AR Path="/57CF2D36/57CF03DE" Ref="D9"  Part="1"
-F 0 "D9" H 5900 3800 50  0000 C CNN
+F 0 "D3" H 5900 3800 50  0000 C CNN
 F 1 "VSLY5850" H 5900 3600 50  0000 C CNN
 F 2 "mouse:LED-5MM_Angle" H 5900 3700 50  0001 C CNN
@@
 AR Path="/57CEFE78/5836B55A" Ref="R7"  Part="1"
 AR Path="/57CF2D36/5836B55A" Ref="R17"  Part="1"
-F 0 "R17" V 5980 4250 50  0000 C CNN
+F 0 "R7" V 5980 4250 50  0000 C CNN
 F 1 "15" V 5900 4250 50  0000 C CNN
 F 2 "Resistors_SMD:R_0805" V 5830 4250 50  0001 C CNN
@@
 AR Path="/57CEFE78/5836B893" Ref="#PWR061"  Part="1"
 AR Path="/57CF2D36/5836B893" Ref="#PWR084"  Part="1"
-F 0 "#PWR084" H 5900 2650 50  0001 C CNN
+F 0 "#PWR061" H 5900 2650 50  0001 C CNN
 F 1 "+5V" H 5900 2940 50  0000 C CNN
 F 2 "" H 5900 2800 50  0000 C CNN
@@
 AR Path="/57CEFE78/5836B8B1" Ref="D2"  Part="1"
 AR Path="/57CF2D36/5836B8B1" Ref="D8"  Part="1"
-F 0 "D8" H 5900 3200 50  0000 C CNN
+F 0 "D2" H 5900 3200 50  0000 C CNN
 F 1 "VSLY5850" H 5900 3000 50  0000 C CNN
 F 2 "mouse:LED-5MM_Angle" H 5900 3100 50  0001 C CNN
@@
 AR Path="/57CEFE78/5836B959" Ref="R8"  Part="1"
 AR Path="/57CF2D36/5836B959" Ref="R18"  Part="1"
-F 0 "R18" V 5580 5050 50  0000 C CNN
+F 0 "R8" V 5580 5050 50  0000 C CNN
 F 1 "10k" V 5500 5050 50  0000 C CNN
 F 2 "Resistors_SMD:R_0402" V 5430 5050 50  0001 C CNN
@@
 AR Path="/57CEFE78/5836B9AB" Ref="#PWR062"  Part="1"
 AR Path="/57CF2D36/5836B9AB" Ref="#PWR085"  Part="1"
-F 0 "#PWR085" H 5500 5050 50  0001 C CNN
+F 0 "#PWR062" H 5500 5050 50  0001 C CNN
 F 1 "GND" H 5500 5150 50  0000 C CNN
 F 2 "" H 5500 5300 50  0000 C CNN

Commit message: 徐々に部品を配置，部品の確認
Parts:
- renumbered R7 to R6, R8 to R7
Changed lines of the file:
@@
 $EndComp
 $Comp
-L GND #PWR060
+L GND #PWR059
 U 1 1 57CF03C0
 P 5900 5300
-AR Path="/57CEFE78/57CF03C0" Ref="#PWR060"  Part="1"
-AR Path="/57CF2D36/57CF03C0" Ref="#PWR083"  Part="1"
-F 0 "#PWR060" H 5900 5050 50  0001 C CNN
+AR Path="/57CEFE78/57CF03C0" Ref="#PWR059"  Part="1"
+AR Path="/57CF2D36/57CF03C0" Ref="#PWR082"  Part="1"
+F 0 "#PWR059" H 5900 5050 50  0001 C CNN
 F 1 "GND" H 5900 5150 50  0000 C CNN
 F 2 "" H 5900 5300 50  0000 C CNN
@@
 IR LED
 $Comp
-L R R7
+L R R6
 U 1 1 5836B55A
 P 5900 4250
-AR Path="/57CEFE78/5836B55A" Ref="R7"  Part="1"
-AR Path="/57CF2D36/5836B55A" Ref="R17"  Part="1"
-F 0 "R7" V 5980 4250 50  0000 C CNN
+AR Path="/57CEFE78/5836B55A" Ref="R6"  Part="1"
+AR Path="/57CF2D36/5836B55A" Ref="R16"  Part="1"
+F 0 "R6" V 5980 4250 50  0000 C CNN
 F 1 "15" V 5900 4250 50  0000 C CNN
 F 2 "Resistors_SMD:R_0805" V 5830 4250 50  0001 C CNN
@@
 	5900 4100 5900 3900
 $Comp
-L +5V #PWR061
+L +5V #PWR060
 U 1 1 5836B893
 P 5900 2800
-AR Path="/57CEFE78/5836B893" Ref="#PWR061"  Part="1"
-AR Path="/57CF2D36/5836B893" Ref="#PWR084"  Part="1"
-F 0 "#PWR061" H 5900 2650 50  0001 C CNN
+AR Path="/57CEFE78/5836B893" Ref="#PWR060"  Part="1"
+AR Path="/57CF2D36/5836B893" Ref="#PWR083"  Part="1"
+F 0 "#PWR060" H 5900 2650 50  0001 C CNN
 F 1 "+5V" H 5900 2940 50  0000 C CNN
 F 2 "" H 5900 2800 50  0000 C CNN
@@
 IR_LED_to_IR_LED
 $Comp
-L R R8
+L R R7
 U 1 1 5836B959
 P 5500 5050
-AR Path="/57CEFE78/5836B959" Ref="R8"  Part="1"
-AR Path="/57CF2D36/5836B959" Ref="R18"  Part="1"
-F 0 "R8" V 5580 5050 50  0000 C CNN
+AR Path="/57CEFE78/5836B959" Ref="R7"  Part="1"
+AR Path="/57CF2D36/5836B959" Ref="R17"  Part="1"
+F 0 "R7" V 5580 5050 50  0000 C CNN
 F 1 "10k" V 5500 5050 50  0000 C CNN
 F 2 "Resistors_SMD:R_0402" V 5430 5050 50  0001 C CNN
@@
 Connection ~ 5500 4800
 $Comp
-L GND #PWR062
+L GND #PWR061
 U 1 1 5836B9AB
 P 5500 5300
-AR Path="/57CEFE78/5836B9AB" Ref="#PWR062"  Part="1"
-AR Path="/57CF2D36/5836B9AB" Ref="#PWR085"  Part="1"
-F 0 "#PWR062" H 5500 5050 50  0001 C CNN
+AR Path="/57CEFE78/5836B9AB" Ref="#PWR061"  Part="1"
+AR Path="/57CF2D36/5836B9AB" Ref="#PWR084"  Part="1"
+F 0 "#PWR061" H 5500 5050 50  0001 C CNN
 F 1 "GND" H 5500 5150 50  0000 C CNN
 F 2 "" H 5500 5300 50  0000 C CNN

Commit message: とりあえず全部品を配置
Changed lines of the file:
@@
 AR Path="/57CEFE78/57CF03B8" Ref="Q2"  Part="1"
 AR Path="/57CF2D36/57CF03B8" Ref="Q3"  Part="1"
-F 0 "Q2" H 6100 4850 50  0000 R CNN
+F 0 "Q3" H 6100 4850 50  0000 R CNN
 F 1 "IRFML8244" H 6450 4750 50  0000 R CNN
 F 2 "TO_SOT_Packages_SMD:SOT-23" H 6000 4900 50  0001 C CNN
@@
 AR Path="/57CEFE78/57CF03C0" Ref="#PWR059"  Part="1"
 AR Path="/57CF2D36/57CF03C0" Ref="#PWR082"  Part="1"
-F 0 "#PWR059" H 5900 5050 50  0001 C CNN
+F 0 "#PWR082" H 5900 5050 50  0001 C CNN
 F 1 "GND" H 5900 5150 50  0000 C CNN
 F 2 "" H 5900 5300 50  0000 C CNN
@@
 AR Path="/57CEFE78/57CF03DE" Ref="D3"  Part="1"
 AR Path="/57CF2D36/57CF03DE" Ref="D9"  Part="1"
-F 0 "D3" H 5900 3800 50  0000 C CNN
+F 0 "D9" H 5900 3800 50  0000 C CNN
 F 1 "VSLY5850" H 5900 3600 50  0000 C CNN
 F 2 "mouse:LED-5MM_Angle" H 5900 3700 50  0001 C CNN
@@
 AR Path="/57CEFE78/5836B55A" Ref="R6"  Part="1"
 AR Path="/57CF2D36/5836B55A" Ref="R16"  Part="1"
-F 0 "R6" V 5980 4250 50  0000 C CNN
+F 0 "R16" V 5980 4250 50  0000 C CNN
 F 1 "15" V 5900 4250 50  0000 C CNN
 F 2 "Resistors_SMD:R_0805" V 5830 4250 50  0001 C CNN
@@
 AR Path="/57CEFE78/5836B893" Ref="#PWR060"  Part="1"
 AR Path="/57CF2D36/5836B893" Ref="#PWR083"  Part="1"
-F 0 "#PWR060" H 5900 2650 50  0001 C CNN
+F 0 "#PWR083" H 5900 2650 50  0001 C CNN
 F 1 "+5V" H 5900 2940 50  0000 C CNN
 F 2 "" H 5900 2800 50  0000 C CNN
@@
 AR Path="/57CEFE78/5836B8B1" Ref="D2"  Part="1"
 AR Path="/57CF2D36/5836B8B1" Ref="D8"  Part="1"
-F 0 "D2" H 5900 3200 50  0000 C CNN
+F 0 "D8" H 5900 3200 50  0000 C CNN
 F 1 "VSLY5850" H 5900 3000 50  0000 C CNN
 F 2 "mouse:LED-5MM_Angle" H 5900 3100 50  0001 C CNN
@@
 AR Path="/57CEFE78/5836B959" Ref="R7"  Part="1"
 AR Path="/57CF2D36/5836B959" Ref="R17"  Part="1"
-F 0 "R7" V 5580 5050 50  0000 C CNN
+F 0 "R17" V 5580 5050 50  0000 C CNN
 F 1 "10k" V 5500 5050 50  0000 C CNN
 F 2 "Resistors_SMD:R_0402" V 5430 5050 50  0001 C CNN
@@
 AR Path="/57CEFE78/5836B9AB" Ref="#PWR061"  Part="1"
 AR Path="/57CF2D36/5836B9AB" Ref="#PWR084"  Part="1"
-F 0 "#PWR061" H 5500 5050 50  0001 C CNN
+F 0 "#PWR084" H 5500 5050 50  0001 C CNN
 F 1 "GND" H 5500 5150 50  0000 C CNN
 F 2 "" H 5500 5300 50  0000 C CNN

Commit message: 充電基板を階層に．
Changed lines of the file:
@@
 $Descr A4 11693 8268
 encoding utf-8
-Sheet 5 14
+Sheet 5 15
 Title ""
 Date ""
@@
 AR Path="/57CEFE78/57CF03B8" Ref="Q2"  Part="1"
 AR Path="/57CF2D36/57CF03B8" Ref="Q3"  Part="1"
-F 0 "Q3" H 6100 4850 50  0000 R CNN
+F 0 "Q2" H 6100 4850 50  0000 R CNN
 F 1 "IRFML8244" H 6450 4750 50  0000 R CNN
 F 2 "TO_SOT_Packages_SMD:SOT-23" H 6000 4900 50  0001 C CNN
@@
 AR Path="/57CEFE78/57CF03DE" Ref="D3"  Part="1"
 AR Path="/57CF2D36/57CF03DE" Ref="D9"  Part="1"
-F 0 "D9" H 5900 3800 50  0000 C CNN
+F 0 "D3" H 5900 3800 50  0000 C CNN
 F 1 "VSLY5850" H 5900 3600 50  0000 C CNN
 F 2 "mouse:LED-5MM_Angle" H 5900 3700 50  0001 C CNN
@@
 AR Path="/57CEFE78/5836B55A" Ref="R6"  Part="1"
 AR Path="/57CF2D36/5836B55A" Ref="R16"  Part="1"
-F 0 "R16" V 5980 4250 50  0000 C CNN
+F 0 "R6" V 5980 4250 50  0000 C CNN
 F 1 "15" V 5900 4250 50  0000 C CNN
 F 2 "Resistors_SMD:R_0805" V 5830 4250 50  0001 C CNN
@@
 AR Path="/57CEFE78/5836B8B1" Ref="D2"  Part="1"
 AR Path="/57CF2D36/5836B8B1" Ref="D8"  Part="1"
-F 0 "D8" H 5900 3200 50  0000 C CNN
+F 0 "D2" H 5900 3200 50  0000 C CNN
 F 1 "VSLY5850" H 5900 3000 50  0000 C CNN
 F 2 "mouse:LED-5MM_Angle" H 5900 3100 50  0001 C CNN
@@
 AR Path="/57CEFE78/5836B959" Ref="R7"  Part="1"
 AR Path="/57CF2D36/5836B959" Ref="R17"  Part="1"
-F 0 "R17" V 5580 5050 50  0000 C CNN
+F 0 "R7" V 5580 5050 50  0000 C CNN
 F 1 "10k" V 5500 5050 50  0000 C CNN
 F 2 "Resistors_SMD:R_0402" V 5430 5050 50  0001 C CNN
