File: kicad/Motor.sch (KiCad schematic (older format))
At the start: 3 parts, among them P1 MT-ENC, U2 DRV8835

Commit message: フットプリント調整
Changed lines of the file:
@@
 AR Path="/57CA18F6/57CA1E0F" Ref="U2"  Part="1"
 AR Path="/57CA507C/57CA1E0F" Ref="U3"  Part="1"
-F 0 "U3" H 5350 4550 60  0000 L CNN
+F 0 "U2" H 5350 4550 60  0000 L CNN
 F 1 "DRV8835" H 5950 4550 60  0000 L CNN
 F 2 "mouse:DRV8835" H 5400 4350 60  0001 C CNN
@@
 AR Path="/57CA18F6/57CA1E2A" Ref="#PWR012"  Part="1"
 AR Path="/57CA507C/57CA1E2A" Ref="#PWR021"  Part="1"
-F 0 "#PWR021" H 5600 3550 50  0001 C CNN
+F 0 "#PWR012" H 5600 3550 50  0001 C CNN
 F 1 "+3.3V" H 5600 3840 50  0000 C CNN
 F 2 "" H 5600 3700 50  0000 C CNN
@@
 AR Path="/57CA18F6/57CA1E38" Ref="#PWR013"  Part="1"
 AR Path="/57CA507C/57CA1E38" Ref="#PWR022"  Part="1"
-F 0 "#PWR022" H 5700 4550 50  0001 C CNN
+F 0 "#PWR013" H 5700 4550 50  0001 C CNN
 F 1 "GND" H 5700 4650 50  0000 C CNN
 F 2 "" H 5700 4800 50  0000 C CNN
@@
 AR Path="/57CA18F6/57CA1E3F" Ref="#PWR014"  Part="1"
 AR Path="/57CA507C/57CA1E3F" Ref="#PWR023"  Part="1"
-F 0 "#PWR023" H 6000 4550 50  0001 C CNN
+F 0 "#PWR014" H 6000 4550 50  0001 C CNN
 F 1 "GND" H 6000 4650 50  0000 C CNN
 F 2 "" H 6000 4800 50  0000 C CNN
@@
 AR Path="/57CA18F6/57CA1E46" Ref="#PWR015"  Part="1"
 AR Path="/57CA507C/57CA1E46" Ref="#PWR024"  Part="1"
-F 0 "#PWR024" H 5100 4550 50  0001 C CNN
+F 0 "#PWR015" H 5100 4550 50  0001 C CNN
 F 1 "GND" H 5100 4650 50  0000 C CNN
 F 2 "" H 5100 4800 50  0000 C CNN
@@
 AR Path="/57CA18F6/57CA1E4E" Ref="P1"  Part="1"
 AR Path="/57CA507C/57CA1E4E" Ref="P2"  Part="1"
-F 0 "P2" H 5850 3300 50  0000 C CNN
+F 0 "P1" H 5850 3300 50  0000 C CNN
 F 1 "MT-ENC" H 5850 2900 50  0000 C CNN
 F 2 "Pin_Headers:Pin_Header_Straight_2x03" H 5850 1900 50  0001 C CNN
@@
 AR Path="/57CA18F6/57CA1E57" Ref="#PWR016"  Part="1"
 AR Path="/57CA507C/57CA1E57" Ref="#PWR025"  Part="1"
-F 0 "#PWR025" H 5500 3050 50  0001 C CNN
+F 0 "#PWR016" H 5500 3050 50  0001 C CNN
 F 1 "GND" H 5500 3150 50  0000 C CNN
 F 2 "" H 5500 3300 50  0000 C CNN
@@
 AR Path="/57CA18F6/57CA1E65" Ref="#PWR017"  Part="1"
 AR Path="/57CA507C/57CA1E65" Ref="#PWR026"  Part="1"
-F 0 "#PWR026" H 6200 2750 50  0001 C CNN
+F 0 "#PWR017" H 6200 2750 50  0001 C CNN
 F 1 "+5V" H 6200 3040 50  0000 C CNN
 F 2 "" H 6200 2900 50  0000 C CNN
@@
 AR Path="/57CA18F6/57CCEFE0" Ref="C12"  Part="1"
 AR Path="/57CA507C/57CCEFE0" Ref="C13"  Part="1"
-F 0 "C13" H 4125 4350 50  0000 L CNN
+F 0 "C12" H 4125 4350 50  0000 L CNN
 F 1 "0.1u" H 4125 4150 50  0000 L CNN
 F 2 "Capacitors_SMD:C_0402" H 4138 4100 50  0001 C CNN
@@
 AR Path="/57CA18F6/57CCF032" Ref="#PWR018"  Part="1"
 AR Path="/57CA507C/57CCF032" Ref="#PWR027"  Part="1"
-F 0 "#PWR027" H 4100 3550 50  0001 C CNN
+F 0 "#PWR018" H 4100 3550 50  0001 C CNN
 F 1 "+3.3V" H 4100 3840 50  0000 C CNN
 F 2 "" H 4100 3700 50  0000 C CNN
@@
 AR Path="/57CA18F6/57CCF046" Ref="#PWR019"  Part="1"
 AR Path="/57CA507C/57CCF046" Ref="#PWR028"  Part="1"
-F 0 "#PWR028" H 4100 4550 50  0001 C CNN
+F 0 "#PWR019" H 4100 4550 50  0001 C CNN
 F 1 "GND" H 4100 4650 50  0000 C CNN
 F 2 "" H 4100 4800 50  0000 C CNN
@@
 AR Path="/57CA18F6/57CD5BEE" Ref="#PWR020"  Part="1"
 AR Path="/57CA507C/57CD5BEE" Ref="#PWR029"  Part="1"
-F 0 "#PWR029" H 5900 3550 50  0001 C CNN
+F 0 "#PWR020" H 5900 3550 50  0001 C CNN
 F 1 "+BATT" H 5900 3840 50  0000 C CNN
 F 2 "" H 5900 3700 50  0000 C CNN

Commit message: 徐々に部品を配置，部品の確認
Parts:
- P1: footprint Pin_Headers:Pin_Header_Straight_2x03 -> mouse:1717
- renumbered C12 to C10
Changed lines of the file:
@@
 AR Path="/57CA18F6/57CA1E0F" Ref="U2"  Part="1"
 AR Path="/57CA507C/57CA1E0F" Ref="U3"  Part="1"
-F 0 "U2" H 5350 4550 60  0000 L CNN
+F 0 "U3" H 5350 4550 60  0000 L CNN
 F 1 "DRV8835" H 5950 4550 60  0000 L CNN
 F 2 "mouse:DRV8835" H 5400 4350 60  0001 C CNN
@@
 Connection ~ 5000 4100
 $Comp
-L +3.3V #PWR012
+L +3.3V #PWR010
 U 1 1 57CA1E2A
 P 5600 3700
-AR Path="/57CA18F6/57CA1E2A" Ref="#PWR012"  Part="1"
-AR Path="/57CA507C/57CA1E2A" Ref="#PWR021"  Part="1"
-F 0 "#PWR012" H 5600 3550 50  0001 C CNN
+AR Path="/57CA18F6/57CA1E2A" Ref="#PWR010"  Part="1"
+AR Path="/57CA507C/57CA1E2A" Ref="#PWR019"  Part="1"
+F 0 "#PWR019" H 5600 3550 50  0001 C CNN
 F 1 "+3.3V" H 5600 3840 50  0000 C CNN
 F 2 "" H 5600 3700 50  0000 C CNN
@@
 	5900 3700 5900 3800
 $Comp
-L GND #PWR013
+L GND #PWR011
 U 1 1 57CA1E38
 P 5700 4800
-AR Path="/57CA18F6/57CA1E38" Ref="#PWR013"  Part="1"
-AR Path="/57CA507C/57CA1E38" Ref="#PWR022"  Part="1"
-F 0 "#PWR013" H 5700 4550 50  0001 C CNN
+AR Path="/57CA18F6/57CA1E38" Ref="#PWR011"  Part="1"
+AR Path="/57CA507C/57CA1E38" Ref="#PWR020"  Part="1"
+F 0 "#PWR020" H 5700 4550 50  0001 C CNN
 F 1 "GND" H 5700 4650 50  0000 C CNN
 F 2 "" H 5700 4800 50  0000 C CNN
@@
 	5700 4800 5700 4700
 $Comp
-L GND #PWR014
+L GND #PWR012
 U 1 1 57CA1E3F
 P 6000 4800
-AR Path="/57CA18F6/57CA1E3F" Ref="#PWR014"  Part="1"
-AR Path="/57CA507C/57CA1E3F" Ref="#PWR023"  Part="1"
-F 0 "#PWR014" H 6000 4550 50  0001 C CNN
+AR Path="/57CA18F6/57CA1E3F" Ref="#PWR012"  Part="1"
+AR Path="/57CA507C/57CA1E3F" Ref="#PWR021"  Part="1"
+F 0 "#PWR021" H 6000 4550 50  0001 C CNN
 F 1 "GND" H 6000 4650 50  0000 C CNN
 F 2 "" H 6000 4800 50  0000 C CNN
@@
 	6000 4800 6000 4700
 $Comp
-L GND #PWR015
+L GND #PWR013
 U 1 1 57CA1E46
 P 5100 4800
-AR Path="/57CA18F6/57CA1E46" Ref="#PWR015"  Part="1"
-AR Path="/57CA507C/57CA1E46" Ref="#PWR024"  Part="1"
-F 0 "#PWR015" H 5100 4550 50  0001 C CNN
+AR Path="/57CA18F6/57CA1E46" Ref="#PWR013"  Part="1"
+AR Path="/57CA507C/57CA1E46" Ref="#PWR022"  Part="1"
+F 0 "#PWR022" H 5100 4550 50  0001 C CNN
 F 1 "GND" H 5100 4650 50  0000 C CNN
 F 2 "" H 5100 4800 50  0000 C CNN
@@
 AR Path="/57CA18F6/57CA1E4E" Ref="P1"  Part="1"
 AR Path="/57CA507C/57CA1E4E" Ref="P2"  Part="1"
-F 0 "P1" H 5850 3300 50  0000 C CNN
+F 0 "P2" H 5850 3300 50  0000 C CNN
 F 1 "MT-ENC" H 5850 2900 50  0000 C CNN
-F 2 "Pin_Headers:Pin_Header_Straight_2x03" H 5850 1900 50  0001 C CNN
+F 2 "mouse:1717" H 5850 1900 50  0001 C CNN
 F 3 "" H 5850 1900 50  0000 C CNN
 	1    5850 3100
@@
 $EndComp
 $Comp
-L GND #PWR016
+L GND #PWR014
 U 1 1 57CA1E57
 P 5500 3300
-AR Path="/57CA18F6/57CA1E57" Ref="#PWR016"  Part="1"
-AR Path="/57CA507C/57CA1E57" Ref="#PWR025"  Part="1"
-F 0 "#PWR016" H 5500 3050 50  0001 C CNN
+AR Path="/57CA18F6/57CA1E57" Ref="#PWR014"  Part="1"
+AR Path="/57CA507C/57CA1E57" Ref="#PWR023"  Part="1"
+F 0 "#PWR023" H 5500 3050 50  0001 C CNN
 F 1 "GND" H 5500 3150 50  0000 C CNN
 F 2 "" H 5500 3300 50  0000 C CNN
@@
 	6300 3200 6100 3200
 $Comp
-L +5V #PWR017
+L +5V #PWR015
 U 1 1 57CA1E65
 P 6200 2900
-AR Path="/57CA18F6/57CA1E65" Ref="#PWR017"  Part="1"
-AR Path="/57CA507C/57CA1E65" Ref="#PWR026"  Part="1"
-F 0 "#PWR017" H 6200 2750 50  0001 C CNN
+AR Path="/57CA18F6/57CA1E65" Ref="#PWR015"  Part="1"
+AR Path="/57CA507C/57CA1E65" Ref="#PWR024"  Part="1"
+F 0 "#PWR024" H 6200 2750 50  0001 C CNN
 F 1 "+5V" H 6200 3040 50  0000 C CNN
 F 2 "" H 6200 2900 50  0000 C CNN
@@
 Motor and Encoder
 $Comp
-L C C12
+L C C10
 U 1 1 57CCEFE0
 P 4100 4250
-AR Path="/57CA18F6/57CCEFE0" Ref="C12"  Part="1"
-AR Path="/57CA507C/57CCEFE0" Ref="C13"  Part="1"
-F 0 "C12" H 4125 4350 50  0000 L CNN
+AR Path="/57CA18F6/57CCEFE0" Ref="C10"  Part="1"
+AR Path="/57CA507C/57CCEFE0" Ref="C11"  Part="1"
+F 0 "C11" H 4125 4350 50  0000 L CNN
 F 1 "0.1u" H 4125 4150 50  0000 L CNN
 F 2 "Capacitors_SMD:C_0402" H 4138 4100 50  0001 C CNN
@@
 $EndComp
 $Comp
-L +3.3V #PWR018
+L +3.3V #PWR016
 U 1 1 57CCF032
 P 4100 3700
-AR Path="/57CA18F6/57CCF032" Ref="#PWR018"  Part="1"
-AR Path="/57CA507C/57CCF032" Ref="#PWR027"  Part="1"
-F 0 "#PWR018" H 4100 3550 50  0001 C CNN
+AR Path="/57CA18F6/57CCF032" Ref="#PWR016"  Part="1"
+AR Path="/57CA507C/57CCF032" Ref="#PWR025"  Part="1"
+F 0 "#PWR025" H 4100 3550 50  0001 C CNN
 F 1 "+3.3V" H 4100 3840 50  0000 C CNN
 F 2 "" H 4100 3700 50  0000 C CNN
@@
 $EndComp
 $Comp
-L GND #PWR019
+L GND #PWR017
 U 1 1 57CCF046
 P 4100 4800
-AR Path="/57CA18F6/57CCF046" Ref="#PWR019"  Part="1"
-AR Path="/57CA507C/57CCF046" Ref="#PWR028"  Part="1"
-F 0 "#PWR019" H 4100 4550 50  0001 C CNN
+AR Path="/57CA18F6/57CCF046" Ref="#PWR017"  Part="1"
+AR Path="/57CA507C/57CCF046" Ref="#PWR026"  Part="1"
+F 0 "#PWR026" H 4100 4550 50  0001 C CNN
 F 1 "GND" H 4100 4650 50  0000 C CNN
 F 2 "" H 4100 4800 50  0000 C CNN
@@
 	4100 4400 4100 4800
 $Comp
-L +BATT #PWR020
+L +BATT #PWR018
 U 1 1 57CD5BEE
 P 5900 3700
-AR Path="/57CA18F6/57CD5BEE" Ref="#PWR020"  Part="1"
-AR Path="/57CA507C/57CD5BEE" Ref="#PWR029"  Part="1"
-F 0 "#PWR020" H 5900 3550 50  0001 C CNN
+AR Path="/57CA18F6/57CD5BEE" Ref="#PWR018"  Part="1"
+AR Path="/57CA507C/57CD5BEE" Ref="#PWR027"  Part="1"
+F 0 "#PWR027" H 5900 3550 50  0001 C CNN
 F 1 "+BATT" H 5900 3840 50  0000 C CNN
 F 2 "" H 5900 3700 50  0000 C CNN

Commit message: 充電基板を階層に．
Changed lines of the file:
@@
 $Descr A4 11693 8268
 encoding utf-8
-Sheet 2 14
+Sheet 2 15
 Title ""
 Date ""
@@
 AR Path="/57CA18F6/57CA1E0F" Ref="U2"  Part="1"
 AR Path="/57CA507C/57CA1E0F" Ref="U3"  Part="1"
-F 0 "U3" H 5350 4550 60  0000 L CNN
+F 0 "U2" H 5350 4550 60  0000 L CNN
 F 1 "DRV8835" H 5950 4550 60  0000 L CNN
 F 2 "mouse:DRV8835" H 5400 4350 60  0001 C CNN
@@
 AR Path="/57CA18F6/57CA1E4E" Ref="P1"  Part="1"
 AR Path="/57CA507C/57CA1E4E" Ref="P2"  Part="1"
-F 0 "P2" H 5850 3300 50  0000 C CNN
+F 0 "P1" H 5850 3300 50  0000 C CNN
 F 1 "MT-ENC" H 5850 2900 50  0000 C CNN
 F 2 "mouse:1717" H 5850 1900 50  0001 C CNN
@@
 AR Path="/57CA18F6/57CCEFE0" Ref="C10"  Part="1"
 AR Path="/57CA507C/57CCEFE0" Ref="C11"  Part="1"
-F 0 "C11" H 4125 4350 50  0000 L CNN
+F 0 "C10" H 4125 4350 50  0000 L CNN
 F 1 "0.1u" H 4125 4150 50  0000 L CNN
 F 2 "Capacitors_SMD:C_0402" H 4138 4100 50  0001 C CNN
