File: kicad/Motor.sch (KiCad schematic (older format))
At the start: 3 parts, among them P1 MT-ENC, U2 DRV8835

Commit message: 新基板，部品を配置
Changed lines of the file:
@@
 AR Path="/57CA18F6/57CA1E0F" Ref="U2"  Part="1"
 AR Path="/57CA507C/57CA1E0F" Ref="U3"  Part="1"
-F 0 "U2" H 5350 4550 60  0000 L CNN
+F 0 "U3" H 5350 4550 60  0000 L CNN
 F 1 "DRV8835" H 5950 4550 60  0000 L CNN
 F 2 "mouse:DRV8835" H 5400 4350 60  0001 C CNN
@@
 AR Path="/57CA18F6/57CA1E4E" Ref="P1"  Part="1"
 AR Path="/57CA507C/57CA1E4E" Ref="P2"  Part="1"
-F 0 "P1" H 5850 3300 50  0000 C CNN
+F 0 "P2" H 5850 3300 50  0000 C CNN
 F 1 "MT-ENC" H 5850 2900 50  0000 C CNN
 F 2 "mouse:1717" H 5850 1900 50  0001 C CNN
@@
 AR Path="/57CA18F6/57CCEFE0" Ref="C10"  Part="1"
 AR Path="/57CA507C/57CCEFE0" Ref="C11"  Part="1"
-F 0 "C10" H 4125 4350 50  0000 L CNN
+F 0 "C11" H 4125 4350 50  0000 L CNN
 F 1 "0.1u" H 4125 4150 50  0000 L CNN
 F 2 "Capacitors_SMD:C_0402" H 4138 4100 50  0001 C CNN
