File: kicad/Mouse-01.sch (KiCad schematic (older format))
At the start: 13 parts, among them SW1 RESET, U1 STM32F405RGTx

Commit message: フットプリント調整
Parts:
- SW1: footprint module:SKRPACE010 -> mouse:SW_PUSH
Changed lines of the file:
@@
 F 0 "SW1" H 3900 3550 50  0000 C CNN
 F 1 "RESET" H 3900 2950 50  0000 C CNN
-F 2 "module:SKRPACE010" V 3850 3250 60  0001 C CNN
+F 2 "mouse:SW_PUSH" V 3850 3250 60  0001 C CNN
 F 3 "" V 3850 3250 60  0000 C CNN
 	1    3900 3300

Commit message: 徐々に部品を配置，部品の確認
Parts:
- removed C6, C7: 22u, Capacitors_SMD:C_0805, symbol C_Small
- renumbered C8 to C6, C9 to C7, C10 to C8, C11 to C9
Connections:
- net MT-IN-R-1: now also U1.29 (I2C2_SCL/I2S2_CK/SPI2_SCK/TIM2_CH3/USART3_TX/USB_OTG_HS_ULPI_D3/PB10); no longer U1.16 (ADC1_IN2/ADC2_IN2/ADC3_IN2/TIM2_CH3/TIM5_CH3/TIM9_CH1/USART2_TX/PA2)
- net MT-IN-R-2: now also U1.30 (ADC1_EXTI11/ADC2_EXTI11/ADC3_EXTI11/I2C2_SDA/TIM2_CH4/USART3_RX/USB_OTG_HS_ULPI_D4/PB11); no longer U1.17 (ADC1_IN3/ADC2_IN3/ADC3_IN3/TIM2_CH4/TIM5_CH4/TIM9_CH2/USART2_RX/USB_OTG_HS_ULPI_D0/PA3)
- net SPEAKER: now also U1.61 (CAN1_RX/I2C1_SCL/SDIO_D4/TIM10_CH1/TIM4_CH3/PB8); no longer U1.62 (CAN1_TX/DAC_EXTI9/I2C1_SDA/I2S2_WS/SDIO_D5/SPI2_NSS/TIM11_CH1/TIM4_CH4/PB9)
- net UART-RX: now also U1.17 (ADC1_IN3/ADC2_IN3/ADC3_IN3/TIM2_CH4/TIM5_CH4/TIM9_CH2/USART2_RX/USB_OTG_HS_ULPI_D0/PA3); no longer U1.43 (TIM1_CH3/USART1_RX/USB_OTG_FS_ID/PA10)
- net UART-TX: now also U1.16 (ADC1_IN2/ADC2_IN2/ADC3_IN2/TIM2_CH3/TIM5_CH3/TIM9_CH1/USART2_TX/PA2); no longer U1.42 (DAC_EXTI9/I2C3_SMBA/TIM1_CH2/USART1_TX/USB_OTG_FS_VBUS/PA9)
Changed lines of the file:
@@
 $EndComp
 $Comp
-L C_Small C11
+L C_Small C9
 U 1 1 57C91C59
 P 4500 4800
-F 0 "C11" H 4510 4870 50  0000 L CNN
+F 0 "C9" H 4510 4870 50  0000 L CNN
 F 1 "2.2u" H 4510 4720 50  0000 L CNN
 F 2 "Capacitors_SMD:C_0603" H 4500 4800 50  0001 C CNN
@@
 $EndComp
 $Comp
-L C_Small C10
+L C_Small C8
 U 1 1 57C928EA
 P 4500 4550
-F 0 "C10" H 4510 4620 50  0000 L CNN
+F 0 "C8" H 4510 4620 50  0000 L CNN
 F 1 "2.2u" H 4510 4470 50  0000 L CNN
 F 2 "Capacitors_SMD:C_0603" H 4500 4550 50  0001 C CNN
@@
 Text GLabel 10400 800  2    50   Input ~ 0
 MT-IN-L-1
-Text GLabel 10400 1000 2    50   Input ~ 0
+Text GLabel 10400 3500 2    50   Input ~ 0
 MT-IN-R-1
 Text GLabel 10400 900  2    50   Input ~ 0
 MT-IN-L-2
-Text GLabel 10400 1100 2    50   Input ~ 0
+Text GLabel 10400 3600 2    50   Input ~ 0
 MT-IN-R-2
 $Comp
@@
 $EndComp
 $Comp
-L C_Small C8
+L C_Small C6
 U 1 1 57CDB4B2
 P 4500 2300
-F 0 "C8" H 4510 2370 50  0000 L CNN
+F 0 "C6" H 4510 2370 50  0000 L CNN
 F 1 "0.1u" H 4510 2220 50  0000 L CNN
 F 2 "Capacitors_SMD:C_0402" H 4500 2300 50  0001 C CNN
@@
 RESET
 $Comp
-L C C9
+L C C7
 U 1 1 57CDEB3C
 P 4600 3300
-F 0 "C9" H 4625 3400 50  0000 L CNN
+F 0 "C7" H 4625 3400 50  0000 L CNN
 F 1 "0.1u" H 4625 3200 50  0000 L CNN
 F 2 "Capacitors_SMD:C_0402" H 4638 3150 50  0001 C CNN
@@
 Text GLabel 10400 2800 2    50   Input ~ 0
 SWO
-Text GLabel 10400 1800 2    50   Input ~ 0
+Text GLabel 10400 1100 2    50   Input ~ 0
 UART-RX
-Text GLabel 10400 1700 2    50   Input ~ 0
+Text GLabel 10400 1000 2    50   Input ~ 0
 UART-TX
 Text GLabel 1200 2100 0    50   Input ~ 0
@@
 Text GLabel 10400 2500 2    50   Input ~ 0
 BUTTON
-Text GLabel 10400 3400 2    50   Input ~ 0
+Text GLabel 10400 3300 2    50   Input ~ 0
 SPEAKER
 $Comp
@@
 NoConn ~ 10300 2300
 NoConn ~ 10300 2700
-NoConn ~ 10300 3300
-NoConn ~ 10300 3500
-NoConn ~ 10300 3600
 NoConn ~ 10300 3700
 NoConn ~ 10300 3800
@@
 Wire Wire Line
 	4300 1100 4300 2600
-Wire Wire Line
-	3900 1700 4400 1700
 Connection ~ 4300 2000
 Wire Wire Line
@@
 	10300 4500 10400 4500
 Wire Wire Line
-	10400 1700 10300 1700
-Wire Wire Line
-	10300 1800 10400 1800
+	10400 1000 10300 1000
+Wire Wire Line
+	10300 1100 10400 1100
 Wire Wire Line
 	10400 3900 10300 3900
@@
 	10400 5000 10300 5000
 Wire Wire Line
-	10400 3400 10300 3400
+	10400 3300 10300 3300
 Wire Wire Line
 	10300 3200 10400 3200
@@
 	10300 1200 10400 1200
 Wire Wire Line
-	10400 1100 10300 1100
-Wire Wire Line
-	10300 1000 10400 1000
+	10400 3600 10300 3600
+Wire Wire Line
+	10300 3500 10400 3500
 Wire Wire Line
 	10400 900  10300 900
@@
 Text Notes 700  800  0    100  ~ 0
 Main
-$Comp
-L C_Small C7
-U 1 1 583842DF
-P 4100 2300
-F 0 "C7" H 4110 2370 50  0000 L CNN
-F 1 "22u" H 4110 2220 50  0000 L CNN
-F 2 "Capacitors_SMD:C_0805" H 4100 2300 50  0001 C CNN
-F 3 "" H 4100 2300 50  0000 C CNN
-	1    4100 2300
-	1    0    0    -1
-$EndComp
-$Comp
-L C_Small C6
-U 1 1 58384648
-P 3900 2300
-F 0 "C6" H 3910 2370 50  0000 L CNN
-F 1 "22u" H 3910 2220 50  0000 L CNN
-F 2 "Capacitors_SMD:C_0805" H 3900 2300 50  0001 C CNN
-F 3 "" H 3900 2300 50  0000 C CNN
-	1    3900 2300
-	1    0    0    -1
-$EndComp
-$Comp
-L GND #PWR010
-U 1 1 58384747
-P 4100 2600
-F 0 "#PWR010" H 4100 2350 50  0001 C CNN
-F 1 "GND" H 4100 2450 50  0000 C CNN
-F 2 "" H 4100 2600 50  0000 C CNN
-F 3 "" H 4100 2600 50  0000 C CNN
-	1    4100 2600
-	1    0    0    -1
-$EndComp
-$Comp
-L GND #PWR011
-U 1 1 58384839
-P 3900 2600
-F 0 "#PWR011" H 3900 2350 50  0001 C CNN
-F 1 "GND" H 3900 2450 50  0000 C CNN
-F 2 "" H 3900 2600 50  0000 C CNN
-F 3 "" H 3900 2600 50  0000 C CNN
-	1    3900 2600
-	1    0    0    -1
-$EndComp
-Wire Wire Line
-	4100 2600 4100 2400
-Wire Wire Line
-	3900 2400 3900 2600
-Wire Wire Line
-	3900 1700 3900 2200
-Wire Wire Line
-	4100 2000 4100 2200
-Wire Wire Line
-	4100 2000 4400 2000
+Wire Wire Line
+	4400 1700 4300 1700
+Wire Wire Line
+	4300 2000 4400 2000
+NoConn ~ 10300 3400
+NoConn ~ 10300 1700
+NoConn ~ 10300 1800
 $EndSCHEMATC

Commit message: リポ充電基板を追加
Changed lines of the file:
@@
 $Descr A4 11693 8268
 encoding utf-8
-Sheet 1 13
+Sheet 1 14
 Title ""
 Date ""
@@
 	0    1    1    0
 $EndComp
+$Sheet
+S 4700 6600 800  800
+U 58401A83
+F0 "Charger" 60
+F1 "Charger.sch" 60
+$EndSheet
 $EndSCHEMATC

Commit message: 充電基板を階層に．
Changed lines of the file:
@@
 $Descr A4 11693 8268
 encoding utf-8
-Sheet 1 14
+Sheet 1 15
 Title ""
 Date ""
@@
 $EndComp
 $Sheet
-S 4700 6600 800  800
+S 4700 6600 900  200
 U 58401A83
-F0 "Charger" 60
+F0 "Charger A" 60
 F1 "Charger.sch" 60
 $EndSheet
+$Sheet
+S 4700 7100 900  200
+U 58410148
+F0 "Charger B" 60
+F1 "Charger.sch" 60
+$EndSheet
