File: kicad/Power.sch (KiCad schematic (older format))
At the start: 22 parts, among them P3 Battery_A, P4 Battery_B, Q1 IRLML6402, SW2 Power, U4 LXDC55FAAA-203, U5 REF1933, U6 LT1963ES8

Commit message: 徐々に部品を配置，部品の確認
Parts:
- removed R4: 68, Resistors_SMD:R_0402, symbol R
- added C12: 22u, Capacitors_SMD:C_0805, symbol CP
- R2: value 1k -> 10k
- R5: renamed from R6; value 68 -> 133
- renumbered C14 to C13, C15 to C14, C16 to C15, C17 to C16, C18 to C17, C19 to C18, C20 to C19, C21 to C20, R5 to R4
Connections:
- net +BATT: now also C12.1
- net GND: now also C12.2
- net at U4.11 (FB): now also R5.1
- no-connect marks 1 -> 2
Other:
- moved on the sheet: C13, U4

Commit message: とりあえず全部品を配置
Parts:
- SW2: footprint Pin_Headers:Pin_Header_Straight_1x03 -> mouse:Slide_SW
Changed lines of the file:
@@
 	1    0    0    -1
 $EndComp
-Wire Wire Line
-	9100 2700 9100 3200
 $Comp
 L +BATT #PWR032
@@
 	8800 3200 8800 2800
 Connection ~ 8800 2800
-$Comp
-L CP C15
-U 1 1 57CA26EB
-P 9100 3350
-F 0 "C15" H 9125 3450 50  0000 L CNN
-F 1 "22u" H 9125 3250 50  0000 L CNN
-F 2 "Capacitors_SMD:C_0805" H 9138 3200 50  0001 C CNN
-F 3 "" H 9100 3350 50  0000 C CNN
-	1    9100 3350
-	1    0    0    -1
-$EndComp
-$Comp
-L GND #PWR034
-U 1 1 57CA271B
-P 9100 3700
-F 0 "#PWR034" H 9100 3450 50  0001 C CNN
-F 1 "GND" H 9100 3550 50  0000 C CNN
-F 2 "" H 9100 3700 50  0000 C CNN
-F 3 "" H 9100 3700 50  0000 C CNN
-	1    9100 3700
-	1    0    0    -1
-$EndComp
-Wire Wire Line
-	9100 3700 9100 3500
 Connection ~ 9100 2800
 Wire Wire Line
@@
 	8500 3200 8500 3300
 $Comp
-L +BATT #PWR035
+L +BATT #PWR034
 U 1 1 57CC111A
 P 4800 2700
-F 0 "#PWR035" H 4800 2550 50  0001 C CNN
+F 0 "#PWR034" H 4800 2550 50  0001 C CNN
 F 1 "+BATT" H 4800 2840 50  0000 C CNN
 F 2 "" H 4800 2700 50  0000 C CNN
@@
 $EndComp
 $Comp
-L GND #PWR036
+L GND #PWR035
 U 1 1 57CC113A
 P 3800 3700
-F 0 "#PWR036" H 3800 3450 50  0001 C CNN
+F 0 "#PWR035" H 3800 3450 50  0001 C CNN
 F 1 "GND" H 3800 3550 50  0000 C CNN
 F 2 "" H 3800 3700 50  0000 C CNN
@@
 	3700 2900 4200 2900
 $Comp
-L +5V #PWR037
+L +5V #PWR036
 U 1 1 57CC1940
 P 4100 4400
-F 0 "#PWR037" H 4100 4250 50  0001 C CNN
+F 0 "#PWR036" H 4100 4250 50  0001 C CNN
 F 1 "+5V" H 4100 4540 50  0000 C CNN
 F 2 "" H 4100 4400 50  0000 C CNN
@@
 Connection ~ 4100 4500
 $Comp
-L GND #PWR038
+L GND #PWR037
 U 1 1 57CC1AB4
 P 4900 5300
-F 0 "#PWR038" H 4900 5050 50  0001 C CNN
+F 0 "#PWR037" H 4900 5050 50  0001 C CNN
 F 1 "GND" H 4900 5150 50  0000 C CNN
 F 2 "" H 4900 5300 50  0000 C CNN
@@
 	4900 5300 4900 5100
 $Comp
-L GND #PWR039
+L GND #PWR038
 U 1 1 57CC1B19
 P 4100 5300
-F 0 "#PWR039" H 4100 5050 50  0001 C CNN
+F 0 "#PWR038" H 4100 5050 50  0001 C CNN
 F 1 "GND" H 4100 5150 50  0000 C CNN
 F 2 "" H 4100 5300 50  0000 C CNN
@@
 	4100 5300 4100 5100
 $Comp
-L +3.3VA #PWR040
+L +3.3VA #PWR039
 U 1 1 57CC1D9F
 P 5600 4400
-F 0 "#PWR040" H 5750 4350 50  0001 C CNN
+F 0 "#PWR039" H 5750 4350 50  0001 C CNN
 F 1 "+3.3VA" H 5600 4500 50  0000 C CNN
 F 2 "" H 5600 4400 50  0000 C CNN
@@
 	5600 4500 5400 4500
 $Comp
-L +1.65VA #PWR041
+L +1.65VA #PWR040
 U 1 1 57CC1DFF
 P 6000 4400
-F 0 "#PWR041" H 6150 4350 50  0001 C CNN
+F 0 "#PWR040" H 6150 4350 50  0001 C CNN
 F 1 "+1.65VA" H 6000 4500 50  0000 C CNN
 F 2 "" H 6000 4400 50  0000 C CNN
@@
 $EndComp
 $Comp
-L +5V #PWR042
+L +5V #PWR041
 U 1 1 57CC204D
 P 6600 4400
-F 0 "#PWR042" H 6600 4250 50  0001 C CNN
+F 0 "#PWR041" H 6600 4250 50  0001 C CNN
 F 1 "+5V" H 6600 4540 50  0000 C CNN
 F 2 "" H 6600 4400 50  0000 C CNN
@@
 $EndComp
 $Comp
-L GND #PWR043
+L GND #PWR042
 U 1 1 57CC212C
 P 6600 5300
-F 0 "#PWR043" H 6600 5050 50  0001 C CNN
+F 0 "#PWR042" H 6600 5050 50  0001 C CNN
 F 1 "GND" H 6600 5150 50  0000 C CNN
 F 2 "" H 6600 5300 50  0000 C CNN
@@
 Connection ~ 6900 4500
 $Comp
-L GND #PWR044
+L GND #PWR043
 U 1 1 57CC2261
 P 7600 5300
-F 0 "#PWR044" H 7600 5050 50  0001 C CNN
+F 0 "#PWR043" H 7600 5050 50  0001 C CNN
 F 1 "GND" H 7600 5150 50  0000 C CNN
 F 2 "" H 7600 5300 50  0000 C CNN
@@
 	7700 5200 7700 5100
 $Comp
-L +3.3V #PWR045
+L +3.3V #PWR044
 U 1 1 57CC235F
 P 8500 4400
-F 0 "#PWR045" H 8500 4250 50  0001 C CNN
+F 0 "#PWR044" H 8500 4250 50  0001 C CNN
 F 1 "+3.3V" H 8500 4540 50  0000 C CNN
 F 2 "" H 8500 4400 50  0000 C CNN
@@
 $EndComp
 $Comp
-L GND #PWR046
+L GND #PWR045
 U 1 1 57CC26B1
 P 8500 5300
-F 0 "#PWR046" H 8500 5050 50  0001 C CNN
+F 0 "#PWR045" H 8500 5050 50  0001 C CNN
 F 1 "GND" H 8500 5150 50  0000 C CNN
 F 2 "" H 8500 5300 50  0000 C CNN
@@
 Connection ~ 6000 4600
 $Comp
-L GND #PWR047
+L GND #PWR046
 U 1 1 57CC28D4
 P 5600 5300
-F 0 "#PWR047" H 5600 5050 50  0001 C CNN
+F 0 "#PWR046" H 5600 5050 50  0001 C CNN
 F 1 "GND" H 5600 5150 50  0000 C CNN
 F 2 "" H 5600 5300 50  0000 C CNN
@@
 	5600 5300 5600 5100
 $Comp
-L GND #PWR048
+L GND #PWR047
 U 1 1 57CC2961
 P 6000 5300
-F 0 "#PWR048" H 6000 5050 50  0001 C CNN
+F 0 "#PWR047" H 6000 5050 50  0001 C CNN
 F 1 "GND" H 6000 5150 50  0000 C CNN
 F 2 "" H 6000 5300 50  0000 C CNN
@@
 F 0 "SW2" H 4700 3650 50  0000 C CNN
 F 1 "Power" H 4750 3350 50  0000 C CNN
-F 2 "Pin_Headers:Pin_Header_Straight_1x03" H 4900 3500 50  0001 C CNN
+F 2 "mouse:Slide_SW" H 4900 3500 50  0001 C CNN
 F 3 "" H 4900 3500 50  0000 C CNN
 	1    4900 3500
@@
 $EndComp
 $Comp
-L GND #PWR049
+L GND #PWR048
 U 1 1 57CD3C05
 P 5700 3700
-F 0 "#PWR049" H 5700 3450 50  0001 C CNN
+F 0 "#PWR048" H 5700 3450 50  0001 C CNN
 F 1 "GND" H 5700 3550 50  0000 C CNN
 F 2 "" H 5700 3700 50  0000 C CNN
@@
 	5700 3600 5700 3700
 $Comp
-L +BATT #PWR050
+L +BATT #PWR049
 U 1 1 57CD3CA2
 P 5700 2700
-F 0 "#PWR050" H 5700 2550 50  0001 C CNN
+F 0 "#PWR049" H 5700 2550 50  0001 C CNN
 F 1 "+BATT" H 5700 2840 50  0000 C CNN
 F 2 "" H 5700 2700 50  0000 C CNN
@@
 Connection ~ 5700 3200
 $Comp
-L GND #PWR051
+L GND #PWR050
 U 1 1 57D18DB8
 P 3600 5300
-F 0 "#PWR051" H 3600 5050 50  0001 C CNN
+F 0 "#PWR050" H 3600 5050 50  0001 C CNN
 F 1 "GND" H 3600 5150 50  0000 C CNN
 F 2 "" H 3600 5300 50  0000 C CNN
@@
 $EndComp
 $Comp
-L PWR_FLAG #FLG052
+L PWR_FLAG #FLG051
 U 1 1 57D18DE7
 P 3600 5200
-F 0 "#FLG052" H 3600 5295 50  0001 C CNN
+F 0 "#FLG051" H 3600 5295 50  0001 C CNN
 F 1 "PWR_FLAG" H 3600 5380 50  0000 C CNN
 F 2 "" H 3600 5200 50  0000 C CNN
@@
 	3600 5200 3600 5300
 $Comp
-L PWR_FLAG #FLG053
+L PWR_FLAG #FLG052
 U 1 1 57D1915C
 P 3600 4500
-F 0 "#FLG053" H 3600 4595 50  0001 C CNN
+F 0 "#FLG052" H 3600 4595 50  0001 C CNN
 F 1 "PWR_FLAG" H 3600 4680 50  0000 C CNN
 F 2 "" H 3600 4500 50  0000 C CNN
@@
 $EndComp
 $Comp
-L +BATT #PWR054
+L +BATT #PWR053
 U 1 1 57D1923B
 P 3600 4400
-F 0 "#PWR054" H 3600 4250 50  0001 C CNN
+F 0 "#PWR053" H 3600 4250 50  0001 C CNN
 F 1 "+BATT" H 3600 4540 50  0000 C CNN
 F 2 "" H 3600 4400 50  0000 C CNN
@@
 $EndComp
 $Comp
-L +5V #PWR055
+L +5V #PWR054
 U 1 1 57D009FE
 P 9600 2700
-F 0 "#PWR055" H 9600 2550 50  0001 C CNN
+F 0 "#PWR054" H 9600 2550 50  0001 C CNN
 F 1 "+5V" H 9600 2840 50  0000 C CNN
 F 2 "" H 9600 2700 50  0000 C CNN
@@
 $EndComp
 $Comp
-L GND #PWR056
+L GND #PWR055
 U 1 1 57D00A42
 P 9600 3700
-F 0 "#PWR056" H 9600 3450 50  0001 C CNN
+F 0 "#PWR055" H 9600 3450 50  0001 C CNN
 F 1 "GND" H 9600 3550 50  0000 C CNN
 F 2 "" H 9600 3700 50  0000 C CNN
@@
 $EndComp
 $Comp
-L GND #PWR057
+L GND #PWR056
 U 1 1 5832F827
 P 5400 3700
-F 0 "#PWR057" H 5400 3450 50  0001 C CNN
+F 0 "#PWR056" H 5400 3450 50  0001 C CNN
 F 1 "GND" H 5400 3550 50  0000 C CNN
 F 2 "" H 5400 3700 50  0000 C CNN
@@
 $EndComp
 $Comp
-L GND #PWR058
+L GND #PWR057
 U 1 1 583807ED
 P 6500 3700
-F 0 "#PWR058" H 6500 3450 50  0001 C CNN
+F 0 "#PWR057" H 6500 3450 50  0001 C CNN
 F 1 "GND" H 6500 3550 50  0000 C CNN
 F 2 "" H 6500 3700 50  0000 C CNN
@@
 	9100 2800 8400 2800
 NoConn ~ 5400 3400
+Wire Wire Line
+	9100 2700 9100 3200
+$Comp
+L GND #PWR058
+U 1 1 57CA271B
+P 9100 3700
+F 0 "#PWR058" H 9100 3450 50  0001 C CNN
+F 1 "GND" H 9100 3550 50  0000 C CNN
+F 2 "" H 9100 3700 50  0000 C CNN
+F 3 "" H 9100 3700 50  0000 C CNN
+	1    9100 3700
+	1    0    0    -1
+$EndComp
+Wire Wire Line
+	9100 3700 9100 3500
+$Comp
+L CP C15
+U 1 1 57CA26EB
+P 9100 3350
+F 0 "C15" H 9125 3450 50  0000 L CNN
+F 1 "22u" H 9125 3250 50  0000 L CNN
+F 2 "Capacitors_SMD:C_0805" H 9138 3200 50  0001 C CNN
+F 3 "" H 9100 3350 50  0000 C CNN
+	1    9100 3350
+	1    0    0    -1
+$EndComp
 $EndSCHEMATC

Commit message: ネットリストとデザインルールを更新
Connections:
- net BAT_to_FET: now reaches P3.1 (P1), Q1.2 (S), R3.1
Changed lines of the file:
@@
 	1    0    0    -1
 $EndComp
+Text Label 3800 2900 0    60   ~ 0
+BAT_to_FET
 $EndSCHEMATC

Commit message: ネットリストを更新
Connections:
- net BAT_to_BAT: now reaches P3.2 (P2), P4.1 (P1)
Changed lines of the file:
@@
 Text Label 3800 2900 0    60   ~ 0
 BAT_to_FET
+Text Label 3800 3400 0    60   ~ 0
+BAT_to_BAT
 $EndSCHEMATC
