File: kicad/Power.sch (KiCad schematic (older format))
At the start: 22 parts, among them P3 Battery_A, P4 Battery_B, Q1 IRLML6402, SW2 Power, U4 LXDC55FAAA-203, U5 REF1933, U6 LT1963ES8

Commit message: 自動配線用にdsn吐き出し
Parts:
- removed C16: 0.1u, Capacitors_SMD:C_0402, symbol C
- removed C17, C18: 10u, Capacitors_SMD:C_0603, symbol C
- removed U5: REF1933, TO_SOT_Packages_SMD:SOT-23-5, symbol REF1933
- added R6, R7: 1k, Resistors_SMD:R_0402, symbol R
- renumbered C19 to C16, C20 to C17, U6 to U5
Connections:
- net +1.65VA: now also R6.2, R7.1
- net +3V3: now also R6.1
- net GND: now also R7.2
