File: kicad/UI.sch (KiCad schematic (older format))
At the start: 14 parts, among them Q4 BSS138, SW3 BUTTON

Commit message: 徐々に部品を配置，部品の確認
Parts:
- renumbered C33 to C32, R19 to R18, R20 to R19, R21 to R20, R22 to R21, R23 to R22, R24 to R23
Changed lines of the file:
@@
 $EndComp
 $Comp
-L +3.3V #PWR093
+L +3.3V #PWR092
 U 1 1 57CE7538
 P 4400 3500
-F 0 "#PWR093" H 4400 3350 50  0001 C CNN
+F 0 "#PWR092" H 4400 3350 50  0001 C CNN
 F 1 "+3.3V" H 4400 3640 50  0000 C CNN
 F 2 "" H 4400 3500 50  0000 C CNN
@@
 $EndComp
 $Comp
-L R R24
+L R R23
 U 1 1 57CE757A
 P 4000 4450
-F 0 "R24" V 4080 4450 50  0000 C CNN
+F 0 "R23" V 4080 4450 50  0000 C CNN
 F 1 "10k" V 4000 4450 50  0000 C CNN
 F 2 "Resistors_SMD:R_0402" V 3930 4450 50  0001 C CNN
@@
 $EndComp
 $Comp
-L GND #PWR094
+L GND #PWR093
 U 1 1 57CE7673
 P 4400 4700
-F 0 "#PWR094" H 4400 4450 50  0001 C CNN
+F 0 "#PWR093" H 4400 4450 50  0001 C CNN
 F 1 "GND" H 4400 4550 50  0000 C CNN
 F 2 "" H 4400 4700 50  0000 C CNN
@@
 $EndComp
 $Comp
-L GND #PWR095
+L GND #PWR094
 U 1 1 57CE768B
 P 4000 4700
-F 0 "#PWR095" H 4000 4450 50  0001 C CNN
+F 0 "#PWR094" H 4000 4450 50  0001 C CNN
 F 1 "GND" H 4000 4550 50  0000 C CNN
 F 2 "" H 4000 4700 50  0000 C CNN
@@
 $EndComp
 $Comp
-L GND #PWR096
+L GND #PWR095
 U 1 1 57CE8530
 P 6000 4700
-F 0 "#PWR096" H 6000 4450 50  0001 C CNN
+F 0 "#PWR095" H 6000 4450 50  0001 C CNN
 F 1 "GND" H 6000 4550 50  0000 C CNN
 F 2 "" H 6000 4700 50  0000 C CNN
@@
 $EndComp
 $Comp
-L GND #PWR097
+L GND #PWR096
 U 1 1 57CE8557
 P 6300 4700
-F 0 "#PWR097" H 6300 4450 50  0001 C CNN
+F 0 "#PWR096" H 6300 4450 50  0001 C CNN
 F 1 "GND" H 6300 4550 50  0000 C CNN
 F 2 "" H 6300 4700 50  0000 C CNN
@@
 $EndComp
 $Comp
-L GND #PWR098
+L GND #PWR097
 U 1 1 57CE8577
 P 6600 4700
-F 0 "#PWR098" H 6600 4450 50  0001 C CNN
+F 0 "#PWR097" H 6600 4450 50  0001 C CNN
 F 1 "GND" H 6600 4550 50  0000 C CNN
 F 2 "" H 6600 4700 50  0000 C CNN
@@
 $EndComp
 $Comp
-L GND #PWR099
+L GND #PWR098
 U 1 1 57CE8597
 P 6900 4700
-F 0 "#PWR099" H 6900 4450 50  0001 C CNN
+F 0 "#PWR098" H 6900 4450 50  0001 C CNN
 F 1 "GND" H 6900 4550 50  0000 C CNN
 F 2 "" H 6900 4700 50  0000 C CNN
@@
 	6000 4600 6000 4700
 $Comp
-L R R20
+L R R19
 U 1 1 57CE8600
 P 6000 3950
-F 0 "R20" V 6080 3950 50  0000 C CNN
+F 0 "R19" V 6080 3950 50  0000 C CNN
 F 1 "1k" V 6000 3950 50  0000 C CNN
 F 2 "Resistors_SMD:R_0402" V 5930 3950 50  0001 C CNN
@@
 $EndComp
 $Comp
-L R R21
+L R R20
 U 1 1 57CE8644
 P 6300 3950
-F 0 "R21" V 6380 3950 50  0000 C CNN
+F 0 "R20" V 6380 3950 50  0000 C CNN
 F 1 "1k" V 6300 3950 50  0000 C CNN
 F 2 "Resistors_SMD:R_0402" V 6230 3950 50  0001 C CNN
@@
 $EndComp
 $Comp
-L R R22
+L R R21
 U 1 1 57CE8677
 P 6600 3950
-F 0 "R22" V 6680 3950 50  0000 C CNN
+F 0 "R21" V 6680 3950 50  0000 C CNN
 F 1 "1k" V 6600 3950 50  0000 C CNN
 F 2 "Resistors_SMD:R_0402" V 6530 3950 50  0001 C CNN
@@
 $EndComp
 $Comp
-L R R23
+L R R22
 U 1 1 57CE86AD
 P 6900 3950
-F 0 "R23" V 6980 3950 50  0000 C CNN
+F 0 "R22" V 6980 3950 50  0000 C CNN
 F 1 "1k" V 6900 3950 50  0000 C CNN
 F 2 "Resistors_SMD:R_0402" V 6830 3950 50  0001 C CNN
@@
 	6900 3400 6900 3800
 $Comp
-L GND #PWR0100
+L GND #PWR099
 U 1 1 57CEA2EF
 P 8200 4700
-F 0 "#PWR0100" H 8200 4450 50  0001 C CNN
+F 0 "#PWR099" H 8200 4450 50  0001 C CNN
 F 1 "GND" H 8200 4550 50  0000 C CNN
 F 2 "" H 8200 4700 50  0000 C CNN
@@
 	8200 3700 8200 4000
 $Comp
-L R R19
+L R R18
 U 1 1 57CEA520
 P 8200 3550
-F 0 "R19" V 8280 3550 50  0000 C CNN
+F 0 "R18" V 8280 3550 50  0000 C CNN
 F 1 "10k" V 8200 3550 50  0000 C CNN
 F 2 "Resistors_SMD:R_0402" V 8130 3550 50  0001 C CNN
@@
 $EndComp
 $Comp
-L +3.3V #PWR0101
+L +3.3V #PWR0100
 U 1 1 57CEA571
 P 8200 3300
-F 0 "#PWR0101" H 8200 3150 50  0001 C CNN
+F 0 "#PWR0100" H 8200 3150 50  0001 C CNN
 F 1 "+3.3V" H 8200 3440 50  0000 C CNN
 F 2 "" H 8200 3300 50  0000 C CNN
@@
 Connection ~ 8200 3800
 $Comp
-L C C33
+L C C32
 U 1 1 57CEAAA3
 P 8500 4200
-F 0 "C33" H 8525 4300 50  0000 L CNN
+F 0 "C32" H 8525 4300 50  0000 L CNN
 F 1 "0.1u" H 8525 4100 50  0000 L CNN
 F 2 "Capacitors_SMD:C_0402" H 8538 4050 50  0001 C CNN
@@
 $EndComp
 $Comp
-L GND #PWR0102
+L GND #PWR0101
 U 1 1 57CEAAF6
 P 8500 4700
-F 0 "#PWR0102" H 8500 4450 50  0001 C CNN
+F 0 "#PWR0101" H 8500 4450 50  0001 C CNN
 F 1 "GND" H 8500 4550 50  0000 C CNN
 F 2 "" H 8500 4700 50  0000 C CNN

Commit message: とりあえず全部品を配置
Parts:
- removed R18: 10k, Resistors_SMD:R_0402, symbol R
- renumbered R19 to R18, R20 to R19, R21 to R20, R22 to R21, R23 to R22
Changed lines of the file:
@@
 $EndComp
 $Comp
-L R R23
+L R R22
 U 1 1 57CE757A
 P 4000 4450
-F 0 "R23" V 4080 4450 50  0000 C CNN
+F 0 "R22" V 4080 4450 50  0000 C CNN
 F 1 "10k" V 4000 4450 50  0000 C CNN
 F 2 "Resistors_SMD:R_0402" V 3930 4450 50  0001 C CNN
@@
 	6000 4600 6000 4700
 $Comp
-L R R19
+L R R18
 U 1 1 57CE8600
 P 6000 3950
-F 0 "R19" V 6080 3950 50  0000 C CNN
+F 0 "R18" V 6080 3950 50  0000 C CNN
 F 1 "1k" V 6000 3950 50  0000 C CNN
 F 2 "Resistors_SMD:R_0402" V 5930 3950 50  0001 C CNN
@@
 $EndComp
 $Comp
-L R R20
+L R R19
 U 1 1 57CE8644
 P 6300 3950
-F 0 "R20" V 6380 3950 50  0000 C CNN
+F 0 "R19" V 6380 3950 50  0000 C CNN
 F 1 "1k" V 6300 3950 50  0000 C CNN
 F 2 "Resistors_SMD:R_0402" V 6230 3950 50  0001 C CNN
@@
 $EndComp
 $Comp
-L R R21
+L R R20
 U 1 1 57CE8677
 P 6600 3950
-F 0 "R21" V 6680 3950 50  0000 C CNN
+F 0 "R20" V 6680 3950 50  0000 C CNN
 F 1 "1k" V 6600 3950 50  0000 C CNN
 F 2 "Resistors_SMD:R_0402" V 6530 3950 50  0001 C CNN
@@
 $EndComp
 $Comp
-L R R22
+L R R21
 U 1 1 57CE86AD
 P 6900 3950
-F 0 "R22" V 6980 3950 50  0000 C CNN
+F 0 "R21" V 6980 3950 50  0000 C CNN
 F 1 "1k" V 6900 3950 50  0000 C CNN
 F 2 "Resistors_SMD:R_0402" V 6830 3950 50  0001 C CNN
@@
 Text HLabel 8100 3800 0    60   Input ~ 0
 BUTTON
-Wire Wire Line
-	8100 3800 8500 3800
-Wire Wire Line
-	8200 3700 8200 4000
-$Comp
-L R R18
-U 1 1 57CEA520
-P 8200 3550
-F 0 "R18" V 8280 3550 50  0000 C CNN
-F 1 "10k" V 8200 3550 50  0000 C CNN
-F 2 "Resistors_SMD:R_0402" V 8130 3550 50  0001 C CNN
-F 3 "" H 8200 3550 50  0000 C CNN
-	1    8200 3550
-	1    0    0    -1
-$EndComp
-$Comp
-L +3.3V #PWR0100
-U 1 1 57CEA571
-P 8200 3300
-F 0 "#PWR0100" H 8200 3150 50  0001 C CNN
-F 1 "+3.3V" H 8200 3440 50  0000 C CNN
-F 2 "" H 8200 3300 50  0000 C CNN
-F 3 "" H 8200 3300 50  0000 C CNN
-	1    8200 3300
-	1    0    0    -1
-$EndComp
-Wire Wire Line
-	8200 3300 8200 3400
-Connection ~ 8200 3800
-$Comp
-L C C32
-U 1 1 57CEAAA3
-P 8500 4200
-F 0 "C32" H 8525 4300 50  0000 L CNN
-F 1 "0.1u" H 8525 4100 50  0000 L CNN
-F 2 "Capacitors_SMD:C_0402" H 8538 4050 50  0001 C CNN
-F 3 "" H 8500 4200 50  0000 C CNN
-	1    8500 4200
-	1    0    0    -1
-$EndComp
-$Comp
-L GND #PWR0101
-U 1 1 57CEAAF6
-P 8500 4700
-F 0 "#PWR0101" H 8500 4450 50  0001 C CNN
-F 1 "GND" H 8500 4550 50  0000 C CNN
-F 2 "" H 8500 4700 50  0000 C CNN
-F 3 "" H 8500 4700 50  0000 C CNN
-	1    8500 4700
-	1    0    0    -1
-$EndComp
-Wire Wire Line
-	8500 4700 8500 4350
-Wire Wire Line
-	8500 3800 8500 4050
 $Comp
 L Tactile_SW_4P SW3
@@
 Text Notes 3300 3100 0    100  ~ 0
 User Interface
+Wire Wire Line
+	8200 3800 8200 4000
+Wire Wire Line
+	8100 3800 8500 3800
+$Comp
+L GND #PWR0100
+U 1 1 57CEAAF6
+P 8500 4700
+F 0 "#PWR0100" H 8500 4450 50  0001 C CNN
+F 1 "GND" H 8500 4550 50  0000 C CNN
+F 2 "" H 8500 4700 50  0000 C CNN
+F 3 "" H 8500 4700 50  0000 C CNN
+	1    8500 4700
+	1    0    0    -1
+$EndComp
+$Comp
+L C C32
+U 1 1 583A7129
+P 8500 4250
+F 0 "C32" H 8525 4350 50  0000 L CNN
+F 1 "0.1u" H 8525 4150 50  0000 L CNN
+F 2 "Capacitors_SMD:C_0402" H 8538 4100 50  0001 C CNN
+F 3 "" H 8500 4250 50  0000 C CNN
+	1    8500 4250
+	1    0    0    -1
+$EndComp
+Wire Wire Line
+	8500 4400 8500 4700
+Wire Wire Line
+	8500 3800 8500 4100
+Connection ~ 8200 3800
 $EndSCHEMATC
